File: sensornode/sensornode.kicad_pcb (KiCad board)
At the start: 2 copper layers, 57.6 x 43.9 mm, 29 parts, among them J1 Conn_01x02, J2 Conn_01x06_Male, J3 Conn_01x04_Male, J4 USB_B_Micro, Q1 MMBT3904, U1 ESP-12F, U2 MQ-135, U3 LTC4055, U4 MIC5504-3.3YM5

Commit message: tweaks, add jumper for programming
Parts:
- removed G***: LOGO, logo:diamond
- removed REF** (x2): MountingHole_3.2mm_M3, MountingHole:MountingHole_3.2mm_M3
- moved J4 2.47 mm to (200.2, 97.2)
Connections:
- J4 pad 2: Net-(J4-Pad2) -> (no net)
- J4 pad 3: Net-(J4-Pad3) -> (no net)
- J4 pad 4: Net-(J4-Pad4) -> (no net)
- U1 pad 10: Net-(U1-Pad10) -> (no net)
- U1 pad 11: Net-(U1-Pad11) -> (no net)
- U1 pad 12: Net-(U1-Pad12) -> (no net)
- U1 pad 13: Net-(U1-Pad13) -> (no net)
- U1 pad 14: Net-(U1-Pad14) -> (no net)
- U1 pad 20: Net-(U1-Pad20) -> (no net)
- U1 pad 6: Net-(U1-Pad6) -> (no net)
- U1 pad 7: Net-(U1-Pad7) -> (no net)
- U1 pad 9: Net-(U1-Pad9) -> (no net)
- U2 pad 2: +5V -> (no net)
- U2 pad 3: Net-(U2-Pad3) -> Net-(R10-Pad2)
- U2 pad 5: Net-(U2-Pad5) -> +5V
- U2 pad 7: Net-(R10-Pad2) -> (no net)
- U3 pad 13: Net-(U3-Pad13) -> (no net)
- U3 pad 14: Net-(U3-Pad14) -> (no net)
- U3 pad 15: Net-(U3-Pad15) -> (no net)
- U4 pad 4: Net-(U4-Pad4) -> (no net)
Routing:
- net +5V: track 50.1 -> 65.4 mm
- net Net-(R10-Pad2): track 7.99 -> 17.8 mm
- net GND: track 81.9 -> 81.3 mm

Commit message: add missing libs and footprints, add jumper for programming
Parts:
- added G***: LOGO, logo:diamond, F.Cu at (201.7, 88.2)
- added JP1: SolderJumper_2_Open, Jumper:SolderJumper-2_P1.3mm_Open_Pad1.0x1.5mm, F.Cu at (186.6, 100.4)
Connections:
- J4 pad 2: (no net) -> Net-(J4-Pad2)
- J4 pad 3: (no net) -> Net-(J4-Pad3)
- J4 pad 4: (no net) -> Net-(J4-Pad4)
- U1 pad 10: (no net) -> Net-(U1-Pad10)
- U1 pad 11: (no net) -> Net-(U1-Pad11)
- U1 pad 12: (no net) -> Net-(U1-Pad12)
- U1 pad 13: (no net) -> Net-(U1-Pad13)
- U1 pad 14: (no net) -> Net-(U1-Pad14)
- U1 pad 20: (no net) -> Net-(U1-Pad20)
- U1 pad 4: /~RST -> Net-(JP1-Pad1)
- U1 pad 6: (no net) -> Net-(U1-Pad6)
- U1 pad 7: (no net) -> Net-(U1-Pad7)
- U1 pad 9: (no net) -> Net-(U1-Pad9)
- U2 pad 2: (no net) -> +5V
- U2 pad 3: Net-(R10-Pad2) -> Net-(U2-Pad3)
- U2 pad 5: +5V -> Net-(R10-Pad2)
- U2 pad 7: (no net) -> Net-(U2-Pad7)
- U3 pad 13: (no net) -> Net-(U3-Pad13)
- U3 pad 14: (no net) -> Net-(U3-Pad14)
- U3 pad 15: (no net) -> Net-(U3-Pad15)
- U4 pad 4: (no net) -> Net-(U4-Pad4)
Routing:
- net Net-(JP1-Pad1): track 0.00 -> 36.8 mm, vias 0 -> 2
- net +5V: track 65.4 -> 50.5 mm
- net /~RST: track 28.8 -> 39.7 mm, vias 0 -> 2
- net Net-(R10-Pad2): track 17.8 -> 15.9 mm
- net /SCL: vias 4 -> 3
