File: sensornode/sensornode.kicad_pcb (KiCad board)
At the start: 2 copper layers, 57.6 x 43.9 mm, 30 parts, among them J1 Conn_01x02, J2 Conn_01x06_Male, J3 Conn_01x04_Male, J4 USB_B_Micro, Q1 MMBT3904, U1 ESP-12F, U2 MQ-135, U3 LTC4055, U4 MIC5504-3.3YM5

Commit message: add acpower indication
Parts:
- removed the REF** at (190.8, 62.9)
- removed the REF** at (192.0, 99.2)
- added REF**: MountingHole_3.2mm_M3, MountingHole:MountingHole_3.2mm_M3, F.Cu at (191.0, 62.6)
- added REF**: MountingHole_3.2mm_M3, MountingHole:MountingHole_3.2mm_M3, F.Cu at (192.0, 99.2)
- J1: footprint Connector_JST:JST_EH_B02B-EH-A_1x02_P2.50mm_Vertical -> Connector_JST:JST_PH_B2B-PH-K_1x02_P2.00mm_Vertical
- R10: value 1k8 -> 6k8
- moved G*** 0.36 mm to (201.5, 88.0)
Connections:
- J1 pad 1: Net-(J1-Pad1) -> GND
- J1 pad 2: GND -> Net-(J1-Pad2)
- J4 pad 2: Net-(J4-Pad2) -> (no net)
- J4 pad 3: Net-(J4-Pad3) -> (no net)
- J4 pad 4: Net-(J4-Pad4) -> (no net)
- U1 pad 10: Net-(U1-Pad10) -> (no net)
- U1 pad 11: Net-(U1-Pad11) -> (no net)
- U1 pad 12: Net-(U1-Pad12) -> (no net)
- U1 pad 13: Net-(U1-Pad13) -> (no net)
- U1 pad 14: Net-(U1-Pad14) -> (no net)
- U1 pad 20: Net-(U1-Pad20) -> /~acpr
- U1 pad 6: Net-(U1-Pad6) -> (no net)
- U1 pad 7: Net-(U1-Pad7) -> (no net)
- U1 pad 9: Net-(U1-Pad9) -> (no net)
- U2 pad 3: Net-(U2-Pad3) -> (no net)
- U2 pad 7: Net-(U2-Pad7) -> (no net)
- U3 pad 13: Net-(U3-Pad13) -> /~acpr
- U3 pad 14: Net-(U3-Pad14) -> (no net)
- U3 pad 15: Net-(U3-Pad15) -> (no net)
- U3 pad 2: Net-(J1-Pad1) -> Net-(J1-Pad2)
- U4 pad 4: Net-(U4-Pad4) -> (no net)
Routing:
- net /~acpr: track 0.00 -> 54.1 mm, vias 0 -> 2
- net Net-(J1-Pad1): track 19.1 -> 0.00 mm, vias 1 -> 0
- net Net-(J1-Pad2): track 0.00 -> 17.4 mm, vias 0 -> 1
- net GND: track 81.3 -> 86.9 mm, vias 5 -> 8
- net +5V: track 50.5 -> 53.6 mm
- net VBUS: track 34.3 -> 37.3 mm
